File: HW/rev_C/MF_badge_2021_rev_C.sch (EAGLE design)
At the start: 81 parts, among them IC1 MCP73831, J1 HRO_31_M_12_USB_C, Q1 SI1308EDL-T1-GE3, Q2 DMG3415U-7, Q3 DMG3415U-7, U1 ESP32-S2-WROOM, U2 AP2112K-3.3, X1 CAPTOUCH_10MM, X2 CAPTOUCH_10MM, X3 CAPTOUCH_10MM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

Commit message: Update
- added schematics for all versions
- added protoshield files
- added files for rev. D
- README update
- removed unnecessary files
Other:
- moved on the sheet: C1, C10, C11, C12, C13, C14, C15, C16, C2, C20, C22, C3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
